File: mooncake_RevA.kicad_pcb (KiCad board)
At the start: 2 copper layers, 45.9 x 48.4 mm, 25 parts, among them U1 MCP23017, X1 Badgelife_shitty_connector

Commit message: Revision B
Parts:
- removed the G*** at (100.0, 100.0)
- added G***: LOGO, mooncake-addon-design:silkscreen, F.Cu at (100.0, 100.0)
- turned C1 to 0 degrees
Routing:
- net Net-(R9-Pad1): track 80.1 -> 37.5 mm, vias 0 -> 2
- net Net-(R10-Pad1): track 69.8 -> 29.3 mm, vias 0 -> 2
- net GND: track 51.8 -> 80.3 mm, vias 4 -> 2
- net scl: track 55.3 -> 35.8 mm, vias 0 -> 2
- net sda: track 48.0 -> 28.8 mm, vias 0 -> 2
- net +3V3: track 41.9 -> 60.1 mm
- net Net-(R1-Pad1): track 40.1 -> 27.2 mm, vias 0 -> 2
- net Net-(R3-Pad1): track 28.7 -> 37.7 mm, vias 0 -> 2
- net Net-(R8-Pad1): track 34.9 -> 29.1 mm, vias 0 -> 2
- net Net-(R2-Pad1): track 34.4 -> 30.1 mm, vias 0 -> 2
- net Net-(R7-Pad1): track 27.8 -> 24.8 mm, vias 0 -> 2
- net Net-(R4-Pad1): track 22.7 -> 20.9 mm, vias 0 -> 2
- net Net-(R6-Pad1): track 18.8 -> 17.8 mm, vias 0 -> 2
- net Net-(R5-Pad1): track 15.5 -> 14.8 mm, vias 0 -> 2
Other:
- board text removed: "Chokity!"
- board text removed: "Design By: d4rkwyng"
- board text removed: "Mooncake Rev. B"
