File: mooncake.kicad_pcb (KiCad board)
At the start: 2 copper layers, 46 x 48.4 mm, 25 parts, among them U1 MCP23017, X1 Badgelife_shitty_connector

Commit message: Issues with EdgeCuts
Parts:
- D1, D10, D2, D3, D4, D5, D6, D7, D8, D9: footprint LEDs:LED_1206_HandSoldering -> mrmeeseeks-addon-lib:LED_1206_HandSoldering_MinSilk
- R1, R10, R2, R3, R4, R5, R6, R7, R8, R9: footprint Resistors_SMD:R_1206_HandSoldering -> mrmeeseeks-addon-lib:R_1206_HandSoldering_NoSilk
Routing:
- net Net-(R9-Pad1): track 0.00 -> 23.1 mm, vias 0 -> 2
- net Net-(D9-Pad2): track 0.00 -> 4.48 mm, vias 0 -> 1
Other:
- board outline removed
- board text added: "#badgelife"
- board text added: "Thank you: AND!XOR SparX"

Commit message: Updated Traces
Gerbers included
Parts:
- C1: footprint Capacitors_SMD:C_0402_NoSilk -> mrmeeseeks-addon-lib:C_0402_NoSilk_NoText
- moved C1 1.32 mm to (100.3, 109.2)
- moved D10 0.66 mm to (109.9, 116.6)
- moved R10 0.66 mm to (109.9, 116.6)
Routing:
- net Net-(R9-Pad1): track 23.1 -> 37.5 mm
- net GND: track 66.3 -> 80.3 mm, vias 8 -> 2
- net Net-(R10-Pad1): track 18.7 -> 29.3 mm
- net +3V3: track 67.6 -> 60.1 mm, vias 6 -> 0
- net sda: track 33.9 -> 28.8 mm
- net scl: track 39.2 -> 35.8 mm
- net Net-(R8-Pad1): track 30.0 -> 29.1 mm
Other:
- board outline added: 45.9 x 48.4 mm

Commit message: Revision B
Parts:
- removed the G*** at (100.0, 100.0)
- added G***: LOGO, design:silkscreen, F.Cu at (100.0, 100.0)
- turned C1 to 180 degrees
Routing:
- net Net-(R9-Pad1): track 37.5 -> 80.1 mm, vias 2 -> 0
- net Net-(R10-Pad1): track 29.3 -> 69.8 mm, vias 2 -> 0
- net GND: track 80.3 -> 51.8 mm, vias 2 -> 4
- net scl: track 35.8 -> 55.3 mm, vias 2 -> 0
- net sda: track 28.8 -> 48.0 mm, vias 2 -> 0
- net +3V3: track 60.1 -> 41.9 mm
- net Net-(R1-Pad1): track 27.2 -> 40.1 mm, vias 2 -> 0
- net Net-(R3-Pad1): track 37.7 -> 28.7 mm, vias 2 -> 0
- net Net-(R8-Pad1): track 29.1 -> 34.9 mm, vias 2 -> 0
- net Net-(R2-Pad1): track 30.1 -> 34.4 mm, vias 2 -> 0
- net Net-(R7-Pad1): track 24.8 -> 27.8 mm, vias 2 -> 0
- net Net-(R4-Pad1): track 20.9 -> 22.7 mm, vias 2 -> 0
- net Net-(R6-Pad1): track 17.8 -> 18.8 mm, vias 2 -> 0
- net Net-(R5-Pad1): track 14.8 -> 15.5 mm, vias 2 -> 0
Other:
- board text added: "Chokity!"
- board text added: "Design By: d4rkwyng"
- board text added: "Mooncake Rev. B"

Commit message: Rev B tweaks
Parts:
- moved D6 3.53 mm to (113.8, 90.2), turned to 325 degrees
- moved R6 3.53 mm to (113.8, 90.2), turned to 325 degrees
- moved D7 1.09 mm to (119.3, 96.0), turned to 298 degrees
- moved R7 1.09 mm to (119.3, 96.0), turned to 298 degrees
- moved D8 0.65 mm to (120.8, 104.3)
- moved R8 0.65 mm to (120.8, 104.3)
Routing:
- net Net-(R6-Pad1): track 18.8 -> 23.8 mm
- net Net-(R3-Pad1): track 28.7 -> 30.2 mm
- net Net-(R2-Pad1): track 34.4 -> 35.9 mm
- net Net-(R7-Pad1): track 27.8 -> 29.0 mm
- net Net-(R4-Pad1): track 22.7 -> 23.9 mm
- net Net-(R8-Pad1): track 34.9 -> 35.9 mm
- net GND: track 51.8 -> 52.8 mm
- net Net-(R1-Pad1): track 40.1 -> 40.9 mm
- net Net-(R5-Pad1): track 15.5 -> 16.0 mm
- net scl: track 55.3 -> 54.8 mm

Commit message: Rev B Updates
Other:
- board text added: "Chookity!"
- board text added: "Thank to: AND!XOR SparX"
- board text removed: "Chokity!"
- board text removed: "Thank you: AND!XOR SparX"
Changed lines of the file:
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@@
     (links 40)
     (no_connects 0)
-    (area 72.009 72.898 129.705101 131.572001)
+    (area 76.950499 75.731299 123.049101 124.306401)
     (thickness 1.6)
     (drawings 277)
@@
   )
   (setup
-    (last_trace_width 0.2)
+    (last_trace_width 0.25)
     (user_trace_width 0.2)
     (user_trace_width 0.5)
@@
     (effects (font (size 0.5 0.5) (thickness 0.125)) (justify mirror))
   )
-  (gr_text Chokity! (at 112.66424 121.65584) (layer B.SilkS)
+  (gr_text Chookity! (at 112.66424 121.65584) (layer B.SilkS)
     (effects (font (size 1 1) (thickness 0.25)) (justify mirror))
   )
-  (gr_text "Design By:\nd4rkwyng" (at 108.4326 111.252) (layer B.SilkS)
-    (effects (font (size 1 1) (thickness 0.25)) (justify mirror))
+  (gr_text "Design By:\nd4rkwyng" (at 104.6099 111.8108) (layer B.SilkS)
+    (effects (font (size 0.75 0.75) (thickness 0.1875)) (justify mirror))
   )
   (gr_line (start 120.6373 94.1959) (end 121.0818 94.9833) (angle 90) (layer Edge.Cuts) (width 0.15))
@@
   (gr_line (start 121.1199 95.0468) (end 121.2596 95.3389) (angle 90) (layer Edge.Cuts) (width 0.15))
   (gr_line (start 121.0818 94.9833) (end 121.1199 95.0468) (angle 90) (layer Edge.Cuts) (width 0.15))
-  (gr_text "Thank you:\nAND!XOR\nSparX" (at 89.8398 111.5568) (layer B.SilkS)
+  (gr_text "Thank to:\nAND!XOR\nSparX" (at 90.1954 110.5281) (layer B.SilkS)
     (effects (font (size 0.75 0.75) (thickness 0.1875)) (justify mirror))
   )
@@
   (segment (start 109.27256 117.33354) (end 110.0328 116.5733) (width 0.25) (layer B.Cu) (net 12))
   (segment (start 107.975615 117.33354) (end 109.27256 117.33354) (width 0.25) (layer B.Cu) (net 12))
-  (segment (start 91.821 97.028) (end 91.821 91.2368) (width 0.2) (layer B.Cu) (net 13) (status 400000))
+  (segment (start 91.821 97.028) (end 91.821 91.2368) (width 0.2) (layer B.Cu) (net 13))
   (segment (start 91.821 91.2368) (end 91.313 90.7288) (width 0.2) (layer B.Cu) (net 13))
   (segment (start 91.313 90.7288) (end 90.87612 90.7288) (width 0.2) (layer B.Cu) (net 13))
@@
   (segment (start 86.68004 112.776) (end 86.68004 113.275385) (width 0.2) (layer B.Cu) (net 13))
   (segment (start 86.68004 113.275385) (end 89.560615 116.15596) (width 0.2) (layer B.Cu) (net 13))
-  (segment (start 93.091 97.028) (end 93.091 90.03284) (width 0.2) (layer B.Cu) (net 14) (status 400000))
+  (segment (start 93.091 97.028) (end 93.091 90.03284) (width 0.2) (layer B.Cu) (net 14))
   (segment (start 93.091 90.03284) (end 92.41028 89.35212) (width 0.2) (layer B.Cu) (net 14))
   (segment (start 92.41028 89.35212) (end 91.65844 89.35212) (width 0.2) (layer B.Cu) (net 14))
@@
   (segment (start 81.897786 107.231746) (end 81.897786 110.345786) (width 0.2) (layer B.Cu) (net 14))
   (segment (start 82.023654 110.345786) (end 81.897786 110.345786) (width 0.25) (layer B.Cu) (net 14) (status 30))
-  (segment (start 94.361 97.028) (end 94.361 89.2556) (width 0.2) (layer B.Cu) (net 15) (status 400000))
+  (segment (start 94.361 97.028) (end 94.361 89.2556) (width 0.2) (layer B.Cu) (net 15))
   (segment (start 94.361 89.2556) (end 94.03588 88.93048) (width 0.2) (layer B.Cu) (net 15))
   (segment (start 94.03588 88.93048) (end 91.51112 88.93048) (width 0.2) (layer B.Cu) (net 15))
@@
   (segment (start 82.34172 95.5548) (end 82.34172 98.221368) (width 0.2) (layer B.Cu) (net 15))
   (segment (start 82.34172 98.221368) (end 78.900704 101.662384) (width 0.2) (layer B.Cu) (net 15))
-  (segment (start 95.631 97.028) (end 95.631 89.79408) (width 0.2) (layer B.Cu) (net 16) (status 400000))
+  (segment (start 95.631 97.028) (end 95.631 89.79408) (width 0.2) (layer B.Cu) (net 16))
   (segment (start 95.631 89.79408) (end 94.26956 88.43264) (width 0.2) (layer B.Cu) (net 16))
   (segment (start 94.26956 88.43264) (end 91.3638 88.43264) (width 0.2) (layer B.Cu) (net 16))

Commit message: Rev B Updates
Other:
- board text added: "Chokity!"
- board text removed: "Chookity!"
Changed lines of the file:
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@@
     (effects (font (size 0.5 0.5) (thickness 0.125)) (justify mirror))
   )
-  (gr_text Chookity! (at 112.66424 121.65584) (layer B.SilkS)
+  (gr_text Chokity! (at 112.66424 121.65584) (layer B.SilkS)
     (effects (font (size 1 1) (thickness 0.25)) (justify mirror))
   )
