File: mooncake_RevC.sch (KiCad schematic (older format))
At the start: 23 parts, among them U1 MCP23017, X1 Badgelife_shitty_connector

Commit message: Revision C
Parts:
- C1: footprint Capacitors_SMD:C_0402_NoSilk -> Capacitors_SMD:C_1206_HandSoldering
- D1, D10, D2, D3, D4, D5, D6, D7, D8, D9: footprint LEDs:LED_1206_HandSoldering -> lib:LED_1206_HandSoldering_MinSilk
- R1, R2, R3, R4, R5, R6, R7, R8, R9: footprint Resistors_SMD:R_1206_HandSoldering -> lib:R_1206_HandSoldering_NoSilk
- R10: footprint (none) -> lib:R_1206_HandSoldering_NoSilk
- U1: footprint SMD_Packages:SOIC-28 -> INTERFACE-MCP23017-E_SOIC28_:SOIC28-1.27-17.9X7.5MM
- X1: footprint mrmeeseeks-addon-lib:Badgelife-Shitty-2x2 -> lib:Badgelife-Shitty-2x2
Changed lines of the file:
@@
 LIBS:valves
 LIBS:badgelife_shitty_connector
-LIBS:mooncake-cache
+LIBS:INTERFACE-MCP23017-E_SOIC28_
 EELAYER 25 0
 EELAYER END
@@
 F 0 "D1" H 2800 2650 50  0000 C CNN
 F 1 "LED" H 2800 2450 50  0000 C CNN
-F 2 "LEDs:LED_1206_HandSoldering" H 2800 2550 50  0001 C CNN
+F 2 "lib:LED_1206_HandSoldering_MinSilk" H 2800 2550 50  0001 C CNN
 F 3 "" H 2800 2550 50  0001 C CNN
 	1    2800 2550
@@
 F 0 "D2" H 2800 2750 50  0000 C CNN
 F 1 "LED" H 2800 2550 50  0000 C CNN
-F 2 "LEDs:LED_1206_HandSoldering" H 2800 2650 50  0001 C CNN
+F 2 "lib:LED_1206_HandSoldering_MinSilk" H 2800 2650 50  0001 C CNN
 F 3 "" H 2800 2650 50  0001 C CNN
 	1    2800 2650
@@
 F 0 "D3" H 2800 2850 50  0000 C CNN
 F 1 "LED" H 2800 2650 50  0000 C CNN
-F 2 "LEDs:LED_1206_HandSoldering" H 2800 2750 50  0001 C CNN
+F 2 "lib:LED_1206_HandSoldering_MinSilk" H 2800 2750 50  0001 C CNN
 F 3 "" H 2800 2750 50  0001 C CNN
 	1    2800 2750
@@
 F 0 "D4" H 2800 2950 50  0000 C CNN
 F 1 "LED" H 2800 2750 50  0000 C CNN
-F 2 "LEDs:LED_1206_HandSoldering" H 2800 2850 50  0001 C CNN
+F 2 "lib:LED_1206_HandSoldering_MinSilk" H 2800 2850 50  0001 C CNN
 F 3 "" H 2800 2850 50  0001 C CNN
 	1    2800 2850
@@
 F 0 "D5" H 2800 3050 50  0000 C CNN
 F 1 "LED" H 2800 2850 50  0000 C CNN
-F 2 "LEDs:LED_1206_HandSoldering" H 2800 2950 50  0001 C CNN
+F 2 "lib:LED_1206_HandSoldering_MinSilk" H 2800 2950 50  0001 C CNN
 F 3 "" H 2800 2950 50  0001 C CNN
 	1    2800 2950
@@
 F 0 "D6" H 2800 3150 50  0000 C CNN
 F 1 "LED" H 2800 2950 50  0000 C CNN
-F 2 "LEDs:LED_1206_HandSoldering" H 2800 3050 50  0001 C CNN
+F 2 "lib:LED_1206_HandSoldering_MinSilk" H 2800 3050 50  0001 C CNN
 F 3 "" H 2800 3050 50  0001 C CNN
 	1    2800 3050
@@
 F 0 "R1" V 3330 2550 50  0000 C CNN
 F 1 "220" V 3250 2550 50  0000 C CNN
-F 2 "Resistors_SMD:R_1206_HandSoldering" V 3180 2550 50  0001 C CNN
+F 2 "lib:R_1206_HandSoldering_NoSilk" V 3180 2550 50  0001 C CNN
 F 3 "" H 3250 2550 50  0001 C CNN
 	1    3250 2550
@@
 F 0 "R2" V 3330 2650 50  0000 C CNN
 F 1 "220" V 3250 2650 50  0000 C CNN
-F 2 "Resistors_SMD:R_1206_HandSoldering" V 3180 2650 50  0001 C CNN
+F 2 "lib:R_1206_HandSoldering_NoSilk" V 3180 2650 50  0001 C CNN
 F 3 "" H 3250 2650 50  0001 C CNN
 	1    3250 2650
@@
 F 0 "R3" V 3330 2750 50  0000 C CNN
 F 1 "220" V 3250 2750 50  0000 C CNN
-F 2 "Resistors_SMD:R_1206_HandSoldering" V 3180 2750 50  0001 C CNN
+F 2 "lib:R_1206_HandSoldering_NoSilk" V 3180 2750 50  0001 C CNN
 F 3 "" H 3250 2750 50  0001 C CNN
 	1    3250 2750
@@
 F 0 "R4" V 3330 2850 50  0000 C CNN
 F 1 "220" V 3250 2850 50  0000 C CNN
-F 2 "Resistors_SMD:R_1206_HandSoldering" V 3180 2850 50  0001 C CNN
+F 2 "lib:R_1206_HandSoldering_NoSilk" V 3180 2850 50  0001 C CNN
 F 3 "" H 3250 2850 50  0001 C CNN
 	1    3250 2850
@@
 F 0 "R5" V 3330 2950 50  0000 C CNN
 F 1 "220" V 3250 2950 50  0000 C CNN
-F 2 "Resistors_SMD:R_1206_HandSoldering" V 3180 2950 50  0001 C CNN
+F 2 "lib:R_1206_HandSoldering_NoSilk" V 3180 2950 50  0001 C CNN
 F 3 "" H 3250 2950 50  0001 C CNN
 	1    3250 2950
@@
 F 0 "R6" V 3330 3050 50  0000 C CNN
 F 1 "220" V 3250 3050 50  0000 C CNN
-F 2 "Resistors_SMD:R_1206_HandSoldering" V 3180 3050 50  0001 C CNN
+F 2 "lib:R_1206_HandSoldering_NoSilk" V 3180 3050 50  0001 C CNN
 F 3 "" H 3250 3050 50  0001 C CNN
 	1    3250 3050
@@
 F 0 "C1" H 5425 3450 50  0000 L CNN
 F 1 "0.1uf" H 5425 3250 50  0000 L CNN
-F 2 "Capacitors_SMD:C_0402_NoSilk" H 5438 3200 50  0001 C CNN
+F 2 "Capacitors_SMD:C_1206_HandSoldering" H 5438 3200 50  0001 C CNN
 F 3 "" H 5400 3350 50  0001 C CNN
 	1    5400 3350
@@
 F 0 "X1" H 5100 5500 60  0000 C CNN
 F 1 "Badgelife_shitty_connector" H 5000 6100 60  0000 C CNN
-F 2 "mrmeeseeks-addon-lib:Badgelife-Shitty-2x2" H 5000 5700 60  0001 C CNN
+F 2 "lib:Badgelife-Shitty-2x2" H 5000 5700 60  0001 C CNN
 F 3 "" H 5000 5700 60  0001 C CNN
 	1    5000 5700
@@
 F 0 "R9" V 3330 3450 50  0000 C CNN
 F 1 "220" V 3250 3450 50  0000 C CNN
-F 2 "Resistors_SMD:R_1206_HandSoldering" V 3180 3450 50  0001 C CNN
+F 2 "lib:R_1206_HandSoldering_NoSilk" V 3180 3450 50  0001 C CNN
 F 3 "" H 3250 3450 50  0001 C CNN
 	1    3250 3450
@@
 F 0 "D9" H 2800 3550 50  0000 C CNN
 F 1 "LED" H 2800 3350 50  0000 C CNN
-F 2 "LEDs:LED_1206_HandSoldering" H 2800 3450 50  0001 C CNN
+F 2 "lib:LED_1206_HandSoldering_MinSilk" H 2800 3450 50  0001 C CNN
 F 3 "" H 2800 3450 50  0001 C CNN
 	1    2800 3450
@@
 F 0 "R10" V 3330 3550 50  0000 C CNN
 F 1 "220" V 3250 3550 50  0000 C CNN
-F 2 "" V 3180 3550 50  0001 C CNN
+F 2 "lib:R_1206_HandSoldering_NoSilk" V 3180 3550 50  0001 C CNN
 F 3 "" H 3250 3550 50  0001 C CNN
 	1    3250 3550
@@
 F 0 "D10" H 2800 3650 50  0000 C CNN
 F 1 "LED" H 2800 3450 50  0000 C CNN
-F 2 "LEDs:LED_1206_HandSoldering" H 2800 3550 50  0001 C CNN
+F 2 "lib:LED_1206_HandSoldering_MinSilk" H 2800 3550 50  0001 C CNN
 F 3 "" H 2800 3550 50  0001 C CNN
 	1    2800 3550
@@
 F 0 "U1" H 3950 4375 50  0000 R CNN
 F 1 "MCP23017" H 3950 4300 50  0000 R CNN
-F 2 "SMD_Packages:SOIC-28" H 4100 2400 50  0001 L CNN
+F 2 "INTERFACE-MCP23017-E_SOIC28_:SOIC28-1.27-17.9X7.5MM" H 4100 2400 50  0001 L CNN
 F 3 "" H 4300 4350 50  0001 C CNN
 	1    4050 3350
@@
 F 0 "R7" V 3330 3150 50  0000 C CNN
 F 1 "220" V 3250 3150 50  0000 C CNN
-F 2 "Resistors_SMD:R_1206_HandSoldering" V 3180 3150 50  0001 C CNN
+F 2 "lib:R_1206_HandSoldering_NoSilk" V 3180 3150 50  0001 C CNN
 F 3 "" H 3250 3150 50  0001 C CNN
 	1    3250 3150
@@
 F 0 "R8" V 3330 3250 50  0000 C CNN
 F 1 "220" V 3250 3250 50  0000 C CNN
-F 2 "Resistors_SMD:R_1206_HandSoldering" V 3180 3250 50  0001 C CNN
+F 2 "lib:R_1206_HandSoldering_NoSilk" V 3180 3250 50  0001 C CNN
 F 3 "" H 3250 3250 50  0001 C CNN
 	1    3250 3250
@@
 F 0 "D7" H 2800 3250 50  0000 C CNN
 F 1 "LED" H 2800 3050 50  0000 C CNN
-F 2 "LEDs:LED_1206_HandSoldering" H 2800 3150 50  0001 C CNN
+F 2 "lib:LED_1206_HandSoldering_MinSilk" H 2800 3150 50  0001 C CNN
 F 3 "" H 2800 3150 50  0001 C CNN
 	1    2800 3150
@@
 F 0 "D8" H 2800 3350 50  0000 C CNN
 F 1 "LED" H 2800 3150 50  0000 C CNN
-F 2 "LEDs:LED_1206_HandSoldering" H 2800 3250 50  0001 C CNN
+F 2 "lib:LED_1206_HandSoldering_MinSilk" H 2800 3250 50  0001 C CNN
 F 3 "" H 2800 3250 50  0001 C CNN
 	1    2800 3250
