File: mooncake_RevC.sch (KiCad schematic (older format))
At the start: 23 parts, among them U1 MCP23017, X1 Badgelife_shitty_connector

Commit message: Fix broken library refs in RevC schematic and add fp-lib-table
mooncake_RevC.sch declared LIBS:INTERFACE-MCP23017-E_SOIC28_, a dangling
reference to U1's footprint name (its F2 field) mistakenly also added as
a symbol library — no such library file exists anywhere in the repo. Same
bug class just fixed in the sibling mrmeeseeks-addon repo. Also corrected
U1 and C1's F2 footprint fields, which pointed at libraries that don't
exist (INTERFACE-MCP23017-E_SOIC28_, Capacitors_SMD) instead of the
lib:SOIC28-1.27-17.9X7.5MM_NoSilk / lib:C_1206_HandSoldering_NoSilk
footprints actually placed on the PCB (confirmed against
mooncake_RevC_BOM.csv, which already listed the correct names).

mooncake_RevC.pro's LibDir pointed at ../mrmeeseeks-addon/lib — a sibling
repo, not this project's own lib/ — breaking on any checkout that doesn't
happen to have that repo cloned next to this one. Pointed it at this
repo's own lib instead.

Added a project-local fp-lib-table (this repo had none) with entries for
every footprint-library nickname actually used by the RevC/RevC_ESO PCBs
(lib, mooncake-design, mrmeeseeks-addon-lib, mooncakes-lib), all pointing
at this repo's own lib/ and design/ directories where the referenced
.kicad_mod files actually live. Verified with kicad-cli 10.0.6: pcb drc
lib_footprint_issues dropped from 28 to 1-2 per board (the remainder is
two footprints — SOIC28-1.27-17.9X7.5MM_NoSilk and
C_1206_HandSoldering_NoSilk — that were only ever embedded in the .kicad_pcb
files and never saved as standalone library files; flagging for Derek
rather than fabricating replacements).

Co-Authored-By: Claude Sonnet 5 <noreply@anthropic.com>
Parts:
- C1: footprint Capacitors_SMD:C_1206_HandSoldering -> lib:C_1206_HandSoldering_NoSilk
- U1: footprint INTERFACE-MCP23017-E_SOIC28_:SOIC28-1.27-17.9X7.5MM -> lib:SOIC28-1.27-17.9X7.5MM_NoSilk
Changed lines of the file:
@@
 LIBS:valves
 LIBS:badgelife_shitty_connector
-LIBS:INTERFACE-MCP23017-E_SOIC28_
 EELAYER 25 0
 EELAYER END
@@
 F 0 "C1" H 5425 3450 50  0000 L CNN
 F 1 "0.1uf" H 5425 3250 50  0000 L CNN
-F 2 "Capacitors_SMD:C_1206_HandSoldering" H 5438 3200 50  0001 C CNN
+F 2 "lib:C_1206_HandSoldering_NoSilk" H 5438 3200 50  0001 C CNN
 F 3 "" H 5400 3350 50  0001 C CNN
 	1    5400 3350
@@
 F 0 "U1" H 3950 4375 50  0000 R CNN
 F 1 "MCP23017" H 3950 4300 50  0000 R CNN
-F 2 "INTERFACE-MCP23017-E_SOIC28_:SOIC28-1.27-17.9X7.5MM" H 4100 2400 50  0001 L CNN
+F 2 "lib:SOIC28-1.27-17.9X7.5MM_NoSilk" H 4100 2400 50  0001 L CNN
 F 3 "" H 4300 4350 50  0001 C CNN
 	1    4050 3350
