File: mooncake_RevC.kicad_pcb (KiCad board)
At the start: 2 copper layers, 45.9 x 48.4 mm, 25 parts, among them U1 MCP23017, X1 Badgelife_shitty_connector

Commit message: Raw Gary Update
Parts:
- added G***: LOGO, mooncake-design:gary_soldermask, B.Cu at (87.4, 103.1)
- C1: footprint Capacitors_SMD:C_1206_HandSoldering -> lib:C_1206_HandSoldering_NoSilk
- U1: footprint INTERFACE-MCP23017-E_SOIC28_:SOIC28-1.27-17.9X7.5MM -> lib:SOIC28-1.27-17.9X7.5MM_NoSilk
- moved U1 0.59 mm to (100.0, 100.0)
- moved X1 0.18 mm to (100.0, 117.0)
Routing:
- net GND: track 117.3 -> 80.7 mm
- net Net-(R10-Pad1): track 65.0 -> 67.5 mm
- net +3V3: track 52.8 -> 54.1 mm
- net Net-(R7-Pad1): track 27.8 -> 27.3 mm
- net Net-(R4-Pad1): track 22.7 -> 22.2 mm
- net Net-(R2-Pad1): track 34.7 -> 34.2 mm
- net sda: track 43.6 -> 43.1 mm
- net scl: track 52.6 -> 52.1 mm
- net Net-(R8-Pad1): track 34.8 -> 34.3 mm
- net Net-(R6-Pad1): track 22.6 -> 22.1 mm
- net Net-(R5-Pad1): track 14.7 -> 14.2 mm
- net Net-(R3-Pad1): track 29.0 -> 28.5 mm
- net Net-(R1-Pad1): track 39.7 -> 39.2 mm

Commit message: The terror that flaps in the night!
Parts:
- added G***: LOGO, mooncake-design:d4rkwyng, B.Cu at (112.3, 104.6)
- added G***: LOGO, mooncake-design:d4rkwyng_solder, B.Cu at (112.3, 104.6)

Commit message: RevC update and ESO version
Routing:
- net GND: track 80.7 -> 83.3 mm
