File: mooncake_RevC_ESO.kicad_pcb (KiCad board)
At the start: 2 copper layers, 45.9 x 48.4 mm, 28 parts, among them U1 MCP23017, X1 Badgelife_shitty_connector

Commit message: RevC update and ESO version
Parts:
- U1: footprint lib:SOIC28-1.27-17.9X7.5MM_NoSilk -> mooncakes-lib:MCP23017-ESS_NoSilk
- turned U1 to 270 degrees
Routing:
- net sda: track 43.1 -> 50.0 mm
- net Net-(R1-Pad1): track 39.2 -> 44.9 mm
- net Net-(R2-Pad1): track 34.2 -> 37.7 mm
- net scl: track 52.1 -> 54.9 mm
- net Net-(R3-Pad1): track 28.5 -> 30.9 mm
- net GND: track 80.7 -> 82.9 mm
- net Net-(R4-Pad1): track 22.2 -> 24.3 mm
- net Net-(R9-Pad1): track 79.4 -> 77.4 mm
- net Net-(R5-Pad1): track 14.2 -> 16.1 mm
- net Net-(R8-Pad1): track 34.3 -> 35.9 mm
- net +3V3: track 54.1 -> 55.6 mm
- net Net-(R7-Pad1): track 27.3 -> 28.5 mm
- net Net-(R10-Pad1): track 67.5 -> 66.3 mm
- net Net-(R6-Pad1): track 22.1 -> 23.0 mm
